File: hardware/peripheral/p2gp2-001.brd (EAGLE design)
At the start: 18 x 31 mm, 3 parts

Commit message: First working model.
Parts:
- added SV2: (no value), con-ml:ML16
- moved LOGO1 13.1 mm to (3.00, 28.0)
Connections:
- net ANLG0: now also SV2.3
- net ANLG1: now also SV2.7
- net ANLG2: now also SV2.11
- net ANLG3: now also SV2.15
- net DTCT0: now also SV2.2
- net DTCT1: now also SV2.6
- net DTCT2: now also SV2.10
- net DTCT3: now also SV2.14
- net GND: now also SV2.1, SV2.13, SV2.5, SV2.9
- net VCC: now also SV2.12, SV2.16, SV2.4, SV2.8
Routing:
- net GND: track 0.00 -> 42.3 mm
- net VCC: track 0.00 -> 42.3 mm
- net DTCT2: track 0.00 -> 8.90 mm
- net ANLG3: track 0.00 -> 8.90 mm
- net ANLG0: track 0.00 -> 8.90 mm
- net DTCT1: track 0.00 -> 8.85 mm
- net ANLG2: track 0.00 -> 8.84 mm
- net DTCT0: track 0.00 -> 8.83 mm
- net DTCT3: track 0.00 -> 8.83 mm
- net ANLG1: track 0.00 -> 8.83 mm
- added copper zone on layer 1, net GND
- added copper zone on layer 16, net GND
Other:
- board text added: "GeekPort II 0.0.1-A"
- board text removed: "GeekPort II 0.0.1"
