File: hardware/peripheral/p2gp2-001.sch (EAGLE design)
At the start: 3 parts

Commit message: First working model.
Parts:
- added SV2: (no value), con-ml:ML16
Connections:
- net ANLG0: now also SV2.3
- net ANLG1: now also SV2.7
- net ANLG2: now also SV2.11
- net ANLG3: now also SV2.15
- net DTCT0: now also SV2.2
- net DTCT1: now also SV2.6
- net DTCT2: now also SV2.10
- net DTCT3: now also SV2.14
- net GND: now also SV2.1, SV2.13, SV2.5, SV2.9
- net VCC: now also SV2.12, SV2.16, SV2.4, SV2.8
Other:
- note removed: "Pineapple -> Switch 1->1 2->4 4->8 8->2"
Changed lines of the file:
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@@
 <part name="SUPPLY3" library="supply2" library_urn="urn:adsk.eagle:library:372" deviceset="VCC" device=""/>
 <part name="U$1" library="pineapple" deviceset="PINEAPPLE450_SILK" device=""/>
+<part name="SV2" library="con-ml" library_urn="urn:adsk.eagle:library:164" deviceset="ML16" device="" package3d_urn="urn:adsk.eagle:package:8674/1"/>
+<part name="SUPPLY2" library="supply2" library_urn="urn:adsk.eagle:library:372" deviceset="VCC" device=""/>
+<part name="SUPPLY4" library="supply2" library_urn="urn:adsk.eagle:library:372" deviceset="GND" device=""/>
 </parts>
 <sheets>
@@
 <plain>
 <text x="218.44" y="20.32" size="1.778" layer="95">Pineapple IIc 2.5.0-RC</text>
-<text x="55.88" y="152.4" size="1.778" layer="97">Pineapple -&gt; Switch
-1-&gt;1
-2-&gt;4
-4-&gt;8
-8-&gt;2</text>
 <text x="139.7" y="101.6" size="1.778" layer="97">GeekPort II
 1: GND
@@
 </instance>
 <instance part="U$1" gate="G$1" x="241.3" y="142.24" smashed="yes"/>
+<instance part="SV2" gate="1" x="66.04" y="101.6" smashed="yes" rot="R180">
+<attribute name="VALUE" x="69.85" y="116.84" size="1.778" layer="96" rot="R180"/>
+<attribute name="NAME" x="69.85" y="90.678" size="1.778" layer="95" rot="R180"/>
+</instance>
+<instance part="SUPPLY2" gate="G$1" x="76.2" y="124.46" smashed="yes">
+<attribute name="VALUE" x="74.295" y="127.635" size="1.778" layer="96"/>
+</instance>
+<instance part="SUPPLY4" gate="GND" x="55.88" y="73.66" smashed="yes">
+<attribute name="VALUE" x="53.975" y="70.485" size="1.778" layer="96"/>
+</instance>
 </instances>
 <busses>
@@
 <junction x="101.6" y="93.98"/>
 </segment>
+<segment>
+<pinref part="SV2" gate="1" pin="1"/>
+<wire x1="58.42" y1="111.76" x2="55.88" y2="111.76" width="0.1524" layer="91"/>
+<wire x1="55.88" y1="111.76" x2="55.88" y2="106.68" width="0.1524" layer="91"/>
+<pinref part="SUPPLY4" gate="GND" pin="GND"/>
+<pinref part="SV2" gate="1" pin="5"/>
+<wire x1="55.88" y1="106.68" x2="55.88" y2="101.6" width="0.1524" layer="91"/>
+<wire x1="55.88" y1="101.6" x2="55.88" y2="96.52" width="0.1524" layer="91"/>
+<wire x1="55.88" y1="96.52" x2="55.88" y2="76.2" width="0.1524" layer="91"/>
+<wire x1="58.42" y1="106.68" x2="55.88" y2="106.68" width="0.1524" layer="91"/>
+<junction x="55.88" y="106.68"/>
+<pinref part="SV2" gate="1" pin="9"/>
+<wire x1="58.42" y1="101.6" x2="55.88" y2="101.6" width="0.1524" layer="91"/>
+<junction x="55.88" y="101.6"/>
+<pinref part="SV2" gate="1" pin="13"/>
+<wire x1="58.42" y1="96.52" x2="55.88" y2="96.52" width="0.1524" layer="91"/>
+<junction x="55.88" y="96.52"/>
+</segment>
 </net>
 <net name="DTCT0" class="0">
@@
 <wire x1="116.84" y1="109.22" x2="132.08" y2="109.22" width="0.1524" layer="91"/>
 <label x="132.08" y="109.22" size="0.8128" layer="95" xref="yes"/>
+</segment>
+<segment>
+<pinref part="SV2" gate="1" pin="2"/>
+<wire x1="73.66" y1="111.76" x2="78.74" y2="111.76" width="0.1524" layer="91"/>
+<label x="78.74" y="111.76" size="0.8128" layer="95" xref="yes"/>
 </segment>
 </net>
@@
 <junction x="124.46" y="101.6"/>
 </segment>
+<segment>
+<pinref part="SV2" gate="1" pin="16"/>
+<wire x1="73.66" y1="93.98" x2="76.2" y2="93.98" width="0.1524" layer="91"/>
+<wire x1="76.2" y1="93.98" x2="76.2" y2="99.06" width="0.1524" layer="91"/>
+<pinref part="SUPPLY2" gate="G$1" pin="VCC"/>
+<pinref part="SV2" gate="1" pin="4"/>
+<wire x1="76.2" y1="99.06" x2="76.2" y2="104.14" width="0.1524" layer="91"/>
+<wire x1="76.2" y1="104.14" x2="76.2" y2="109.22" width="0.1524" layer="91"/>
+<wire x1="76.2" y1="109.22" x2="76.2" y2="121.92" width="0.1524" layer="91"/>
+<wire x1="73.66" y1="109.22" x2="76.2" y2="109.22" width="0.1524" layer="91"/>
+<junction x="76.2" y="109.22"/>
+<pinref part="SV2" gate="1" pin="8"/>
+<wire x1="73.66" y1="104.14" x2="76.2" y2="104.14" width="0.1524" layer="91"/>
+<junction x="76.2" y="104.14"/>
+<pinref part="SV2" gate="1" pin="12"/>
+<wire x1="73.66" y1="99.06" x2="76.2" y2="99.06" width="0.1524" layer="91"/>
+<junction x="76.2" y="99.06"/>
+</segment>
 </net>
 <net name="DTCT1" class="0">
@@
 <label x="132.08" y="104.14" size="0.8128" layer="95" xref="yes"/>
 </segment>
+<segment>
+<pinref part="SV2" gate="1" pin="6"/>
+<wire x1="73.66" y1="106.68" x2="78.74" y2="106.68" width="0.1524" layer="91"/>
+<label x="78.74" y="106.68" size="0.8128" layer="95" xref="yes"/>
+</segment>
 </net>
 <net name="DTCT2" class="0">
@@
 <label x="132.08" y="99.06" size="0.8128" layer="95" xref="yes"/>
 </segment>
+<segment>
+<pinref part="SV2" gate="1" pin="10"/>
+<wire x1="73.66" y1="101.6" x2="78.74" y2="101.6" width="0.1524" layer="91"/>
+<label x="78.74" y="101.6" size="0.8128" layer="95" xref="yes"/>
+</segment>
 </net>
 <net name="DTCT3" class="0">
@@
 <label x="132.08" y="93.98" size="0.8128" layer="95" xref="yes"/>
 </segment>
+<segment>
+<pinref part="SV2" gate="1" pin="14"/>
+<wire x1="73.66" y1="96.52" x2="78.74" y2="96.52" width="0.1524" layer="91"/>
+<label x="78.74" y="96.52" size="0.8128" layer="95" xref="yes"/>
+</segment>
 </net>
 <net name="ANLG0" class="0">
@@
 <label x="96.52" y="106.68" size="0.8128" layer="95" rot="R180" xref="yes"/>
 </segment>
+<segment>
+<pinref part="SV2" gate="1" pin="3"/>
+<wire x1="58.42" y1="109.22" x2="53.34" y2="109.22" width="0.1524" layer="91"/>
+<label x="53.34" y="109.22" size="0.8128" layer="95" rot="R180" xref="yes"/>
+</segment>
 </net>
 <net name="ANLG1" class="0">
@@
 <label x="96.52" y="101.6" size="0.8128" layer="95" rot="R180" xref="yes"/>
 </segment>
+<segment>
+<pinref part="SV2" gate="1" pin="7"/>
+<wire x1="58.42" y1="104.14" x2="53.34" y2="104.14" width="0.1524" layer="91"/>
+<label x="53.34" y="104.14" size="0.8128" layer="95" rot="R180" xref="yes"/>
+</segment>
 </net>
 <net name="ANLG3" class="0">
@@
 <label x="96.52" y="91.44" size="0.8128" layer="95" rot="R180" xref="yes"/>
 </segment>
+<segment>
+<pinref part="SV2" gate="1" pin="15"/>
+<wire x1="58.42" y1="93.98" x2="53.34" y2="93.98" width="0.1524" layer="91"/>
+<label x="53.34" y="93.98" size="0.8128" layer="95" rot="R180" xref="yes"/>
+</segment>
 </net>
 <net name="ANLG2" class="0">
@@
 <label x="96.52" y="96.52" size="0.8128" layer="95" rot="R180" xref="yes"/>
 </segment>
-</net>
+<segment>
+<pinref part="SV2" gate="1" pin="11"/>
+<wire x1="58.42" y1="99.06" x2="53.34" y2="99.06" width="0.1524" layer="91"/>
+<label x="53.34" y="99.06" size="0.8128" layer="95" rot="R180" xref="yes"/>
+</segment>
+</net>
